File: trab/trab.sch (KiCad schematic (older format))
At the start: 17 parts

Commit message: Continuando esquemático
Parts:
- removed Q?: BC337, Package_TO_SOT_THT:TO-92_Inline, symbol Transistor_BJT:BC337
- removed R?: 2200, symbol Device:R
- removed R?: 47000, symbol Device:R
- removed U?: 74HC14, symbol 74xx:74HC14
- added C? (x2): C, symbol Device:C
- added Q? (x2): BC337, Package_TO_SOT_THT:TO-92_Inline, symbol Transistor_BJT:BC337
- added R? (x2): 47k, symbol Device:R
- added R? (x2): 2k2, symbol Device:R
- added R?: 470, symbol Device:R
- added R?: 1M, symbol Device:R
- added U?: 74HC14, symbol 74xx:74HC14
- added U?: LS7366R, symbol trab:LS7366R
- added Y?: 30MHz, symbol Device:Crystal
Connections:
- wire segments 67 -> 89
Other:
- moved on the sheet: Q?

Commit message: Continuando esquemático
Parts:
- removed Q? (x2): BC337, Package_TO_SOT_THT:TO-92_Inline, symbol Transistor_BJT:BC337
- removed R?: 10k, symbol Device:R
- removed R?: 220, symbol Device:R
- removed R? (x2): 470, symbol Device:R
- removed R?: 47000, symbol Device:R
- removed R? (x2): 2k2, symbol Device:R
- removed U?: 4N25, Package_DIP:DIP-6_W7.62mm, symbol Isolator:4N25
- added Q1, Q2: BC337, Package_TO_SOT_THT:TO-92_Inline, symbol trab-cache:BC337
- added R1, R3: 470, symbol Device:R
- added R4, R6: 47k, symbol Device:R
- added U3: GalileoGen2Shield, symbol trab:GalileoGen2Shield
- added U4: MotorEncoder, symbol trab:MotorEncoder
- added U5: MotorDrive, symbol trab:MotorDrive
- C1, C2: renamed from C?; value C -> 22pF
- gave numbers to parts that had none: 14
Connections:
- net labels added: +SAIDA, -SAIDA, A_J1, B_J1, DFLAG_1, EN_1, INDEX_J1, LFLAG_1, MISO, MOSI, MOTOR, SCK, SS_1
- net labels removed: SAIDA+, SAIDA-, external_gnd, pwm
- wire segments 89 -> 115
Other:
- moved on the sheet: Q3, Q4, Q5, Q6, U1A

Commit message: Terminando esquemático
Connections:
- net labels added: INDEX_1, SS
- net labels removed: INDEX_J1, SS_1

Commit message: Versão entregue
Other:
- note added: "10/10/2018"
- note added: "André D. Carneiro, Camilla S. Schmidt e Henrique E. Pchara"
- note added: "Esquemático do projeto final"
Changed lines of the file:
@@
 Text Label 10650 2800 0    50   ~ 0
 INDEX_1
+Text Notes 7100 6700 0    79   ~ 0
+André D. Carneiro, Camilla S. Schmidt e Henrique E. Pchara
+Text Notes 8150 7650 0    50   ~ 0
+10/10/2018
+Text Notes 7400 7500 0    50   ~ 0
+Esquemático do projeto final
 $EndSCHEMATC
