File: esquematico/trab.kicad_pcb (KiCad board)
At the start: 2 copper layers, 11 parts, among them U1 74LS04, U2 74LS08, U3 LS7366R, U4 L298N_2, U5 end, U7 MotorEncoder, U8 GalileoGen2Shield, Y1 30MHz

Commit message: PCB versao 2
Parts:
- C1, C2: footprint Capacitor_THT:C_Rect_L4.6mm_W2.0mm_P2.50mm_MKS02_FKP02 -> Capacitor_THT:C_Rect_L7.0mm_W2.0mm_P5.00mm
- R2: footprint Resistor_THT:R_Axial_DIN0204_L3.6mm_D1.6mm_P7.62mm_Horizontal -> Resistor_THT:R_Axial_DIN0207_L6.3mm_D2.5mm_P10.16mm_Horizontal
- Y1: footprint Crystal:Crystal_C38-LF_D3.0mm_L8.0mm_Vertical -> Crystal:Crystal_AT310_D3.0mm_L10.0mm_Vertical
- moved R2 3.17 mm to (202.6, 62.2)
Routing:
- net /+5V: track 231.2 -> 238.4 mm
- net Net-(C1-Pad1): track 78.8 -> 83.9 mm
- net /INDEX_1: track 111.3 -> 115.8 mm
- net GND: track 488.8 -> 491.6 mm
- net /LFLAG_1: track 152.7 -> 151.6 mm
