File: esquematico/trab.sch (KiCad schematic (older format))
At the start: 25 parts, among them Q1 BC337, Q2 BC337, Q3 TIP122, Q4 TIP122, Q5 TIP122, Q6 TIP122, U1 74HC14, U2 LS7366R, U3 GalileoGen2Shield, U4 MotorEncoder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

Commit message: Layout
Parts:
- removed D1, D2, D3, D4: 1N4148, Diode_THT:D_DO-35_SOD27_P7.62mm_Horizontal, symbol Diode:1N4148
- removed Q1, Q2: BC337, Package_TO_SOT_THT:TO-92_Inline, symbol trab-cache:BC337
- removed Q3, Q4, Q5, Q6: TIP122, Package_TO_SOT_THT:TO-220-3_Vertical, symbol Transistor_BJT:TIP122
- removed R1, R3: 470, symbol Device:R
- removed R4, R5, R6, R7: 47k, symbol Device:R
- removed U1: 74HC14, symbol 74xx:74HC14
- removed U2: LS7366R, symbol trab:LS7366R
- removed U3: GalileoGen2Shield, symbol trab:GalileoGen2Shield
- removed U4: MotorEncoder, symbol trab:MotorEncoder
- removed U5: MotorDrive, symbol trab:MotorDrive
- added U1: 74LS04, lib_footprint:DIP-14_W7.62mm_Socket, symbol 74xx:74LS04
- added U2: 74LS08, lib_footprint:DIP-14_W7.62mm_Socket, symbol 74xx:74LS08
- added U3: LS7366R, Package_DIP:DIP-14_W7.62mm_Socket, symbol micros:LS7366R
- added U4: L298N_2, lib_footprint:krex5, symbol micros:L298N_2
- added U5: end, Connector_Samtec_HLE_THT:Samtec_HLE-116-02-xx-DV-TE_2x08_P2.54mm_Horizontal, symbol micros:end
- added U7: MotorEncoder, lib_footprint:krex4, symbol micros:MotorEncoder
- added U8: GalileoGen2Shield, lib_footprint:galileo, symbol micros:GalileoGen2Shield
- C1, C2: footprint (none) -> Capacitor_THT:C_Rect_L4.6mm_W2.0mm_P2.50mm_MKS02_FKP02
- R2: footprint (none) -> Resistor_THT:R_Axial_DIN0204_L3.6mm_D1.6mm_P7.62mm_Horizontal
- Y1: footprint (none) -> Crystal:Crystal_C38-LF_D3.0mm_L8.0mm_Vertical
Connections:
- net labels added: ELB1, ELB2, ENABLE
- net labels removed: +27V, +SAIDA, -SAIDA
- wire segments 115 -> 78
Other:
- note added: "11/11/2018"
- note added: "Esquemático do projeto final - versão 2"
- note removed: "10/10/2018"
- note removed: "Esquemático do projeto final"

Commit message: PCB versao 2
Parts:
- C1, C2: footprint Capacitor_THT:C_Rect_L4.6mm_W2.0mm_P2.50mm_MKS02_FKP02 -> Capacitor_THT:C_Rect_L7.0mm_W2.0mm_P5.00mm
- R2: footprint Resistor_THT:R_Axial_DIN0204_L3.6mm_D1.6mm_P7.62mm_Horizontal -> Resistor_THT:R_Axial_DIN0207_L6.3mm_D2.5mm_P10.16mm_Horizontal
- Y1: footprint Crystal:Crystal_C38-LF_D3.0mm_L8.0mm_Vertical -> Crystal:Crystal_AT310_D3.0mm_L10.0mm_Vertical
Changed lines of the file:
@@
 F 0 "Y1" V 3254 4631 50  0000 L CNN
 F 1 "30MHz" V 3345 4631 50  0000 L CNN
-F 2 "Crystal:Crystal_C38-LF_D3.0mm_L8.0mm_Vertical" H 3300 4500 50  0001 C CNN
+F 2 "Crystal:Crystal_AT310_D3.0mm_L10.0mm_Vertical" H 3300 4500 50  0001 C CNN
 F 3 "~" H 3300 4500 50  0001 C CNN
 	1    3300 4500
@@
 F 0 "R2" V 3593 4500 50  0000 C CNN
 F 1 "1M" V 3684 4500 50  0000 C CNN
-F 2 "Resistor_THT:R_Axial_DIN0204_L3.6mm_D1.6mm_P7.62mm_Horizontal" V 3730 4500 50  0001 C CNN
+F 2 "Resistor_THT:R_Axial_DIN0207_L6.3mm_D2.5mm_P10.16mm_Horizontal" V 3730 4500 50  0001 C CNN
 F 3 "~" H 3800 4500 50  0001 C CNN
 	1    3800 4500
@@
 F 0 "C1" V 2598 4300 50  0000 C CNN
 F 1 "22pF" V 2689 4300 50  0000 C CNN
-F 2 "Capacitor_THT:C_Rect_L4.6mm_W2.0mm_P2.50mm_MKS02_FKP02" H 2888 4150 50  0001 C CNN
+F 2 "Capacitor_THT:C_Rect_L7.0mm_W2.0mm_P5.00mm" H 2888 4150 50  0001 C CNN
 F 3 "~" H 2850 4300 50  0001 C CNN
 	1    2850 4300
@@
 F 0 "C2" V 2598 4700 50  0000 C CNN
 F 1 "22pF" V 2689 4700 50  0000 C CNN
-F 2 "Capacitor_THT:C_Rect_L4.6mm_W2.0mm_P2.50mm_MKS02_FKP02" H 2888 4550 50  0001 C CNN
+F 2 "Capacitor_THT:C_Rect_L7.0mm_W2.0mm_P5.00mm" H 2888 4550 50  0001 C CNN
 F 3 "~" H 2850 4700 50  0001 C CNN
 	1    2850 4700
@@
 $Comp
 L 74xx:74LS08 U2
-U 3 1 5C0D631F
+U 4 1 5C0D631F
 P 3900 3250
 F 0 "U2" H 3900 3575 50  0000 C CNN
@@
 F 2 "lib_footprint:DIP-14_W7.62mm_Socket" H 3900 3250 50  0001 C CNN
 F 3 "http://www.ti.com/lit/gpn/sn74LS08" H 3900 3250 50  0001 C CNN
-	3    3900 3250
+	4    3900 3250
 	1    0    0    -1
 $EndComp
 $Comp
 L 74xx:74LS04 U1
-U 6 1 5C0D6561
+U 5 1 5C0D6561
 P 3900 2800
 F 0 "U1" H 3900 3117 50  0000 C CNN
@@
 F 2 "lib_footprint:DIP-14_W7.62mm_Socket" H 3900 2800 50  0001 C CNN
 F 3 "http://www.ti.com/lit/gpn/sn74LS04" H 3900 2800 50  0001 C CNN
-	6    3900 2800
+	5    3900 2800
 	1    0    0    -1
 $EndComp
 $Comp
 L 74xx:74LS04 U1
-U 5 1 5C0D662D
+U 6 1 5C0D662D
 P 3850 1850
 F 0 "U1" H 3850 2167 50  0000 C CNN
@@
 F 2 "lib_footprint:DIP-14_W7.62mm_Socket" H 3850 1850 50  0001 C CNN
 F 3 "http://www.ti.com/lit/gpn/sn74LS04" H 3850 1850 50  0001 C CNN
-	5    3850 1850
+	6    3850 1850
 	1    0    0    -1
 $EndComp
 $Comp
 L 74xx:74LS08 U2
-U 4 1 5C0D68CB
+U 3 1 5C0D68CB
 P 4500 2450
 F 0 "U2" H 4500 2775 50  0000 C CNN
@@
 F 2 "lib_footprint:DIP-14_W7.62mm_Socket" H 4500 2450 50  0001 C CNN
 F 3 "http://www.ti.com/lit/gpn/sn74LS08" H 4500 2450 50  0001 C CNN
-	4    4500 2450
-	1    0    0    -1
-$EndComp
+	3    4500 2450
+	1    0    0    -1
+$EndComp
