File: PCB/trab.sch (KiCad schematic (older format))
At the start: 12 parts, among them U1 74LS04, U2 74LS08, U3 LS7366R, U4 L298N, U5 end, U6 MotorDrive, U7 MotorEncoder, U8 GalileoGen2Shield, Y1 30MHz

Commit message: Terminando layout e entrega
Parts:
- removed U4: L298N, symbol micros:L298N
- removed U6: MotorDrive, symbol micros:MotorDrive
- added U4: L298N_2, lib_footprint:krex5, symbol micros:L298N_2
Connections:
- net labels removed: +27V
- wire segments 91 -> 78
Other:
- note added: "11/11/2018"
- note added: "Esquemático do projeto final - versão 2"
- note removed: "11/12/2018"
- note removed: "Esquemático do projeto final\n"
